File: Ethernet_switch_4out/Ethernet_switch_4out.kicad_pcb (KiCad board)
At the start: 4 copper layers, 100 x 100 mm, 224 parts, among them J1 Conn_01x04, J10 RJ45 Abracon ARJM11B1, J11 Conn_01x02, J12 Conn_01x02, J13 Conn_01x02, J14 Jack-DC, J15 Conn_01x06, J2 Conn_01x06, J3 Conn_01x06, J4 USB_C_Receptacle, J5 Conn_01x04, J6 Conn_01x04, J7 RJ45 Abracon ARJM11B1, J8 RJ45 Abracon ARJM11B1, J9 RJ45 Abracon ARJM11B1, SW1 MCU_RESET, SW2 MCU_RESET, SW3 MCU_RESET, U1 ESP32-S3-WROOM-1, U10 MCP6002-xSN, U11 AD5337, U12 XC6206PxxxMR, U13 RT7272B, U2 W5500, U3 RTL8305NB-VB-CG, U4 SRV05-4, U5 CAT24C256, U6 XC6206PxxxMR, U8 INA219AxD, U9 CJ431, Y1 25MHz, Y2 25MHz

Commit message: g
Parts:
- added FID4: Polarity, Symbol:Polarity_Center_Positive_6mm_SilkScreen, F.Cu at (136.1, 70.3)
- moved D37 11.5 mm to (126.2, 80.7)
Routing:
- net GND: track 206.0 -> 265.2 mm, vias 149 -> 748
- net Net-(D37-A): track 10.3 -> 17.7 mm
- net /Cell/Buck_out: track 57.3 -> 64.2 mm
- net /ESP_EN: track 32.2 -> 29.8 mm
Other:
- board text added: "2V5"
- board text added: "3V3"
- board text added: "BOOT"
- board text added: "DAC2"
- board text added: "ENABLE_ESP32"
- board text added: "ENABLE_SWITCH"
- board text added: "GND"
- board text added: "L/R"
- board text added: "RX"
- board text added: "SCK"
- board text added: "SCL"
- board text added: "SD"
- board text added: "SDA"
- board text added: "TX"
- board text added: "WS"
