File: Ethernet_switch_4out/Cell.kicad_sch (KiCad schematic)
At the start: 36 parts, among them J11 Conn_01x02, J14 Jack-DC, J2 Conn_01x06, U10 MCP6002-xSN, U11 AD5337, U13 RT7272B, U8 INA219AxD

Commit message: g
Parts:
- added FID1: Polarity, Symbol:Polarity_Center_Positive_6mm_SilkScreen, symbol Mechanical:Fiducial
Changed lines of the file:
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@@
+    )
+  )
+  (symbol (lib_id "Mechanical:Fiducial") (at 64.77 25.4 0) (unit 1)
+    (in_bom no) (on_board yes) (dnp no) (fields_autoplaced)
+    (property "Reference" "FID1" (at 67.945 24.1299 0)
+      (effects (font (size 1.27 1.27)) (justify left))
+    )
+    (property "Value" "Polarity" (at 67.945 26.6699 0)
+      (effects (font (size 1.27 1.27)) (justify left))
+    )
+    (property "Footprint" "Symbol:Polarity_Center_Positive_6mm_SilkScreen" (at 64.77 25.4 0)
+      (effects (font (size 1.27 1.27)) hide)
+    )
+    (property "Datasheet" "~" (at 64.77 25.4 0)
+      (effects (font (size 1.27 1.27)) hide)
+    )
+    (instances
+      (project "Ethernet_switch_4out"
+        (path "/bc5fbf5d-1090-407a-a25f-f08694d9b93b"
+          (reference "FID1") (unit 1)
+        )
+        (path "/bc5fbf5d-1090-407a-a25f-f08694d9b93b/5cee261c-0256-4f28-8cf6-18c483c8529b"
+          (reference "FID4") (unit 1)
+        )
+      )
+      (project "cross_band_handy_walkie_talkie_ES8388"
+        (path "/cd7625f8-56b3-4b33-9172-cb298da5fb01"
+          (reference "FID1") (unit 1)
+        )
+      )
     )
   )

Commit message: g
Parts:
- added TP2: TestPoint, TestPoint:TestPoint_Pad_D1.0mm, symbol Connector:TestPoint
Connections:
- net DAC1: now also TP2.1
Changed lines of the file:
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@@
   (junction (at 161.29 60.96) (diameter 0) (color 0 0 0 0)
   )
+  (junction (at 120.65 112.395) (diameter 0) (color 0 0 0 0)
+  )
   (junction (at 130.81 60.96) (diameter 0) (color 0 0 0 0)
   )
@@
     (stroke (width 0) (type default))
   )
+  (wire (pts (xy 124.46 112.395) (xy 120.65 112.395))
+    (stroke (width 0) (type default))
+  )
   (wire (pts (xy 137.16 60.96) (xy 152.4 60.96))
     (stroke (width 0) (type default))
@@
     (stroke (width 0) (type default))
   )
-  (wire (pts (xy 120.65 104.14) (xy 120.65 116.84))
+  (wire (pts (xy 120.65 104.14) (xy 120.65 112.395))
     (stroke (width 0) (type default))
   )
@@
   )
   (wire (pts (xy 101.6 73.66) (xy 101.6 74.93))
+    (stroke (width 0) (type default))
+  )
+  (wire (pts (xy 120.65 112.395) (xy 120.65 116.84))
     (stroke (width 0) (type default))
   )
@@
         )
       )
+    )
+  )
+  (symbol (lib_id "Connector:TestPoint") (at 124.46 112.395 270) (unit 1)
+    (in_bom yes) (on_board yes) (dnp no) (fields_autoplaced)
+    (property "Reference" "TP2" (at 130.175 111.76 90)
+      (effects (font (size 1.27 1.27)) (justify left))
+    )
+    (property "Value" "TestPoint" (at 130.175 114.3 90)
+      (effects (font (size 1.27 1.27)) (justify left))
+    )
+    (property "Footprint" "TestPoint:TestPoint_Pad_D1.0mm" (at 124.46 117.475 0)
+      (effects (font (size 1.27 1.27)) hide)
+    )
+    (property "Datasheet" "~" (at 124.46 117.475 0)
+      (effects (font (size 1.27 1.27)) hide)
+    )
+    (pin "1")
+    (instances
+      (project "Ethernet_switch_4out"
+        (path "/bc5fbf5d-1090-407a-a25f-f08694d9b93b"
+          (reference "TP2") (unit 1)
+        )
+        (path "/bc5fbf5d-1090-407a-a25f-f08694d9b93b/6e2bafb1-7e4b-41ce-a220-2f34a277b398"
+          (reference "TP3") (unit 1)
+        )
+        (path "/bc5fbf5d-1090-407a-a25f-f08694d9b93b/5cee261c-0256-4f28-8cf6-18c483c8529b"
+          (reference "TP4") (unit 1)
+        )
+      )

Commit message: e
Parts:
- renumbered C34 to C27, C33 to C52, C35 to C53, C35 to C54, C33 to C56, C33 to C59, C35 to C65, C33 to C66, C35 to C67, C35 to C68, D34 to D36, D34 to D37, FID1 to FID4, J11 to J13, J2 to J15, R72 to R19, R72 to R21, R3 to R67, R3 to R70, R3 to R74, R3 to R75, R3 to R76, R3 to R77, TP2 to TP4
