File: Ethernet_switch_4out/Ethernet_switch_4out.kicad_sch (KiCad schematic)
At the start: 134 parts, among them J1 Conn_01x04, J11 Conn_01x02, J12 Conn_01x02, J2 Conn_01x06, J3 Conn_01x06, J4 USB_C_Receptacle, J5 Conn_01x04, J6 Conn_01x04, SW1 MCU_RESET, SW2 MCU_RESET, SW3 MCU_RESET, U1 ESP32-S3-WROOM-1, U10 MCP6002-xSN, U12 XC6206PxxxMR, U2 W5500, U3 RTL8305NB-VB-CG, U4 SRV05-4, U5 CAT24C256, U6 XC6206PxxxMR, U9 CJ431, Y1 25MHz, Y2 25MHz

Commit message: g
Parts:
- removed C37: 1n, Capacitor_SMD:C_1206_3216Metric, symbol Device:C_Small
- removed J4: USB_C_Receptacle, Connector_USB:USB_C_Receptacle_HRO_TYPE-C-31-M-12, symbol Connector:USB_C_Receptacle
- removed R24: 12k, Resistor_SMD:R_0805_2012Metric, symbol Device:R
- removed R32, R33: 5k1, Resistor_SMD:R_0402_1005Metric, symbol Device:R_Small
- added J4: USB_A, Connector_USB:USB_A_Molex_67643_Horizontal, symbol Connector:USB_A
- added R13: 12k, Resistor_SMD:R_0402_1005Metric, symbol Device:R_Small
- added R18: 10, Resistor_SMD:R_0402_1005Metric, symbol Device:R_Small
- added TP2: TestPoint, TestPoint:TestPoint_Pad_D1.0mm, symbol Connector:TestPoint
- U1: LCSC C2913204 -> (none); site https://jlcpcb.com/partdetail/3198302-ESP32_S3_WROOM_1N8R2/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 -> (none)
Connections:
- net +3V3: now also TP2.1
- net 2V5_RAW: now also R18.2; no longer U9.1 (REF)
- net D+: now also J4.3 (D+)
- net D-: now also J4.2 (D-)
- net GND: now also J4.4 (GND), R13.1
- net VBUS: now also J4.1 (VBUS)
- net at R13.1: now also R13.2
- new net: R18.1, U9.1 (REF)
- no-connect marks 24 -> 15
Other:
- added sheet power (power.kicad_sch)
- moved on the sheet: C14, C15, C57, R13, U10B, U9
