File: Ethernet_switch_4out/Output_port.kicad_sch (KiCad schematic)
At the start: 14 parts, among them J2 RJ45 Abracon ARJM11B1

Commit message: e
Parts:
- renumbered C10 to C38, C10 to C39, C9 to C40, J2 to J7
