File: Ethernet_switch_4out/power.kicad_sch (KiCad schematic)
At the start: 17 parts, among them U7 TX4410

Commit message: xcel fix
Parts:
- U7: value TX4410 -> TX4401
Changed lines of the file:
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@@
       (effects (font (size 1.27 1.27)) (justify left))
     )
-    (property "Value" "TX4410" (at 143.51 52.07 0)
+    (property "Value" "TX4401" (at 143.51 52.07 0)
       (effects (font (size 1.27 1.27)) (justify left))
     )

Commit message: e
Parts:
- renumbered C13 to C37, C14 to C70, C26 to C71, C26 to C72, C13 to C73, C14 to C74, JP1 to JP2, R27 to R78, R27 to R79, TP2 to TP3
